Commit message: adjust params to match real scenarial

File: mr_config/srdf/universal_robots/ur_macro.srdf.xacro (robot description, xacro)
@@ -40,5 +40,5 @@
     </group_state>
     <group_state name="test_1" group="${name}_manipulator">
-      <joint name="${prefix}shoulder_pan_joint" value="0.785" />
+      <joint name="${prefix}shoulder_pan_joint" value="0.0" />
       <joint name="${prefix}shoulder_lift_joint" value="-1.57" />
       <joint name="${prefix}elbow_joint" value="-1.57" />
@@ -47,6 +47,6 @@
       <joint name="${prefix}wrist_3_joint" value="0.0" />
     </group_state>
-        <group_state name="test_2" group="${name}_manipulator">
-      <joint name="${prefix}shoulder_pan_joint" value="3.14" />
+    <group_state name="test_2" group="${name}_manipulator">
+      <joint name="${prefix}shoulder_pan_joint" value="-2.356" />
       <joint name="${prefix}shoulder_lift_joint" value="-1.57" />
       <joint name="${prefix}elbow_joint" value="-1.57" />

File: mr_description/urdf/universal_robots/ur_macro.xacro (robot description, xacro)
@@ -262,5 +262,5 @@
            link/frame) to introduce the necessary rotation over Z (of pi rad).
       -->
-      <origin xyz="0 0 0" rpy="0 0 ${pi}" />
+      <origin xyz="0 0 0" rpy="0 0 0" />
     </joint>
     <joint name="${prefix}shoulder_pan_joint" type="revolute">
@@ -350,5 +350,5 @@
            the UR controller.
       -->
-      <origin xyz="0 0 0" rpy="0 0 ${pi}"/>
+      <origin xyz="0 0 0" rpy="0 0 0"/>
       <parent link="${prefix}base_link"/>
       <child link="${prefix}base"/>

Commit message: config setting for bin picking task

File: mr_config/srdf/universal_robots/ur_macro.srdf.xacro (robot description, xacro)
@@ -5,5 +5,5 @@
     A URDF file must exist for this robot as well, where the joints and the links that are referenced are defined
 -->
-  <xacro:macro name="ur_srdf" params="name prefix">
+  <xacro:macro name="ur_srdf" params="name prefix tool_tip">
     <!--GROUPS - Representation of a set of joints and links. This can be useful for specifying DOF to plan for, defining arms, end effectors, etc-->
     <!--LINKS - When a link is specified, the parent joint of that link (if it exists) is automatically included-->
@@ -12,5 +12,5 @@
     <!--SUBGROUPS - Groups can also be formed by referencing to already defined group names-->
     <group name="${name}_manipulator">
-      <chain base_link="${prefix}base_link" tip_link="${prefix}tool_tip" />
+      <chain base_link="${prefix}base_link" tip_link="${prefix}${tool_tip}" />
     </group>
     <!--GROUP STATES - Purpose - Define a named state for a particular group, in terms of joint values. This is useful to define states like 'folded arms'-->

File: mr_config/srdf/universal_robots/ur_tool_changeable.srdf.xacro (robot description, xacro)
@@ -6,4 +6,4 @@
   <xacro:arg name="prefix" default="" />
   <xacro:include filename="$(find mr_config)/srdf/universal_robots/ur_macro.srdf.xacro"/>
-  <xacro:ur_srdf name="$(arg name)" prefix="$(arg prefix)" tool_tip="tool_tip"/>
+  <xacro:ur_srdf name="$(arg name)" prefix="$(arg prefix)" tool_tip="suction_tool_tip"/>
 </robot>

File: mr_description/urdf/tools/hiwin_gripper.xacro (robot description, xacro)
@@ -7,5 +7,5 @@
                 rpy="0 0 0" />
             <geometry>
-                <mesh filename="package://ur_description/meshes/tool/tool_no_suctoin_1.stl" />
+                <mesh filename="file://$(find mr_description)/meshes/tool/tool_no_suctoin.stl" />
             </geometry>
         </visual>
@@ -15,5 +15,5 @@
                 rpy="0 0 0" />
             <geometry>
-                <mesh filename="package://ur_description/meshes/tool/tool_no_suctoin_1.stl" />
+                <mesh filename="file://$(find mr_description)/meshes/tool/tool_no_suctoin.stl" />
             </geometry>
         </collision>
