Commit message: update urdf

File: mr_description/urdf/universal_robots/ur_tool_changeable.urdf.xacro (robot description, xacro)
@@ -122,5 +122,5 @@
   </joint>
   <joint name="$(arg prefix)base-azure" type="fixed">
-    <origin xyz="0.205016 -0.559936 0.869848" rpy="-3.042109 1.5225345 -1.4807895"/>
+    <origin xyz="0.199425791 -0.590375233 0.856386688" rpy="1.4863183 1.5578821  3.0648614"/>
     <parent link="$(arg prefix)base_link"/>
     <child link="camera_base"/>

Commit message: new scene and tool config

File: mr_description/urdf/universal_robots/ur_tool_changeable.urdf.xacro (robot description, xacro)
@@ -112,5 +112,5 @@
   </joint>
   <joint name="$(arg prefix)suction_tool" type="fixed">
-    <origin xyz="0.02 0 0.363" rpy="0 0 0"/>
+    <origin xyz="0.02 0 0.323" rpy="0 0 0"/>
     <parent link="$(arg prefix)tool_base"/>
     <child link="$(arg prefix)suction_tool_tip"/>

Commit message: longer tool tip

File: mr_description/urdf/universal_robots/ur_tool_changeable.urdf.xacro (robot description, xacro)
@@ -112,5 +112,5 @@
   </joint>
   <joint name="$(arg prefix)suction_tool" type="fixed">
-    <origin xyz="0.02 0 0.323" rpy="0 0 0"/>
+    <origin xyz="0.02 0 0.33" rpy="0 0 0"/>
     <parent link="$(arg prefix)tool_base"/>
     <child link="$(arg prefix)suction_tool_tip"/>

Commit message: update box mesh

File: mr_description/urdf/universal_robots/ur_tool_changeable.urdf.xacro (robot description, xacro)
@@ -117,10 +117,10 @@
   </joint>
   <joint name="$(arg prefix)base-d405" type="fixed">
-    <origin xyz="0.312 -0.134 -0.04" rpy="-1.0443611 0.0053113 -1.5836444"/>
+    <origin xyz="0.24816342683501683 -0.15421478088509458 -0.09905737640547956" rpy="-1.006184 0.0013119 -1.5359343"/>
     <parent link="$(arg prefix)base_link"/>
     <child link="$(arg prefix)d405_link"/>
   </joint>
   <joint name="$(arg prefix)base-azure" type="fixed">
-    <origin xyz="0.199425791 -0.590375233 0.856386688" rpy="1.4863183 1.5578821  3.0648614"/>
+    <origin xyz="0.199425791 -0.590375233 0.866386688" rpy="1.4863183 1.5578821  3.0648614"/>
     <parent link="$(arg prefix)base_link"/>
     <child link="camera_base"/>
